File: VFD_Clock_LD8035.sch (KiCad schematic (older format))
At the start: 22 parts, among them J1 Conn_01x04, J2 Conn_01x04, J3 CONN_01X05, SW1 SW_Push, SW2 SW_Push, U2 TD62783, U3 TD62783

Commit message: Add documentation
Parts:
- V1, V2, V3, V4, V5, V6: footprint VFD:LD8035E -> VFD:LD8035E_Castellated
Changed lines of the file:
@@
 F 0 "V1" H 9400 1175 60  0000 C CNN
 F 1 "ld8035e" H 9225 1375 60  0000 C CNN
-F 2 "VFD:LD8035E" H 8600 1350 60  0001 C CNN
+F 2 "VFD:LD8035E_Castellated" H 8600 1350 60  0001 C CNN
 F 3 "" H 8600 1350 60  0000 C CNN
 	1    8600 1300
@@
 F 0 "V2" H 9400 2375 60  0000 C CNN
 F 1 "ld8035e" H 9225 2575 60  0000 C CNN
-F 2 "VFD:LD8035E" H 8600 2550 60  0001 C CNN
+F 2 "VFD:LD8035E_Castellated" H 8600 2550 60  0001 C CNN
 F 3 "" H 8600 2550 60  0000 C CNN
 	1    8600 2500
@@
 F 0 "V3" H 9400 3575 60  0000 C CNN
 F 1 "ld8035e" H 9225 3775 60  0000 C CNN
-F 2 "VFD:LD8035E" H 8600 3750 60  0001 C CNN
+F 2 "VFD:LD8035E_Castellated" H 8600 3750 60  0001 C CNN
 F 3 "" H 8600 3750 60  0000 C CNN
 	1    8600 3700
@@
 F 0 "V4" H 9400 4825 60  0000 C CNN
 F 1 "ld8035e" H 9225 5025 60  0000 C CNN
-F 2 "VFD:LD8035E" H 8600 5000 60  0001 C CNN
+F 2 "VFD:LD8035E_Castellated" H 8600 5000 60  0001 C CNN
 F 3 "" H 8600 5000 60  0000 C CNN
 	1    8600 4950
@@
 F 0 "V5" H 11250 1175 60  0000 C CNN
 F 1 "ld8035e" H 11075 1375 60  0000 C CNN
-F 2 "VFD:LD8035E" H 10450 1350 60  0001 C CNN
+F 2 "VFD:LD8035E_Castellated" H 10450 1350 60  0001 C CNN
 F 3 "" H 10450 1350 60  0000 C CNN
 	1    10450 1300
@@
 F 0 "V6" H 11250 2375 60  0000 C CNN
 F 1 "ld8035e" H 11075 2575 60  0000 C CNN
-F 2 "VFD:LD8035E" H 10450 2550 60  0001 C CNN
+F 2 "VFD:LD8035E_Castellated" H 10450 2550 60  0001 C CNN
 F 3 "" H 10450 2550 60  0000 C CNN
 	1    10450 2500

Commit message: update
Parts:
- removed J3: CONN_01X05, Pin_Headers:Pin_Header_Straight_1x05_Pitch2.54mm, symbol VFD_Clock_LD8035-rescue:CONN_01X05
- added J3: DS3231_RTC_MODULE, VFD:DS3231_RPi_Module, symbol VFDClock_LD8035:DS3231_RTC_MODULE
Connections:
- net +5V: now also J3.5 (VCC)
- net GND: now also J3.1 (GND)
- net SCL: now also J3.3 (SCL)
- net SDA: now also J3.2 (NC)
Changed lines of the file:
@@
 EESchema Schematic File Version 4
 LIBS:VFD_Clock_LD8035-cache
-EELAYER 26 0
+EELAYER 29 0
 EELAYER END
 $Descr A4 11693 8268
@@
 	1    10700 2000
 	0    -1   1    0
-$EndComp
-$Comp
-L VFD_Clock_LD8035-rescue:CONN_01X05 J3
-U 1 1 5AC3CB54
-P 3800 6950
-F 0 "J3" H 3800 7250 50  0000 C CNN
-F 1 "CONN_01X05" V 3900 6950 50  0000 C CNN
-F 2 "Pin_Headers:Pin_Header_Straight_1x05_Pitch2.54mm" H 3800 6950 50  0001 C CNN
-F 3 "" H 3800 6950 50  0001 C CNN
-	1    3800 6950
-	1    0    0    -1
 $EndComp
 Text Notes 3550 6500 0    60   ~ 0
@@
 L VFD_Clock_LD8035-rescue:GND #PWR012
 U 1 1 5AC419D7
-P 3450 7300
-F 0 "#PWR012" H 3450 7050 50  0001 C CNN
-F 1 "GND" H 3450 7150 50  0000 C CNN
-F 2 "" H 3450 7300 50  0001 C CNN
-F 3 "" H 3450 7300 50  0001 C CNN
-	1    3450 7300
-	1    0    0    -1
-$EndComp
-$Comp
-L VFD_Clock_LD8035-rescue:+5V #PWR013
-U 1 1 5AC42D74
-P 3450 6600
-F 0 "#PWR013" H 3450 6450 50  0001 C CNN
-F 1 "+5V" H 3450 6740 50  0000 C CNN
-F 2 "" H 3450 6600 50  0001 C CNN
-F 3 "" H 3450 6600 50  0001 C CNN
-	1    3450 6600
-	1    0    0    -1
-$EndComp
-Wire Wire Line
-	3600 6750 3200 6750
-Wire Wire Line
-	3600 6850 3200 6850
-Wire Wire Line
-	3600 6950 3200 6950
-Wire Wire Line
-	3600 7050 3450 7050
-Wire Wire Line
-	3450 7050 3450 6600
-Wire Wire Line
-	3600 7150 3450 7150
-Wire Wire Line
-	3450 7150 3450 7300
-Text Label 3200 6750 0    60   ~ 0
-DS
-Text Label 3200 6850 0    60   ~ 0
+P 3250 7500
+F 0 "#PWR012" H 3250 7250 50  0001 C CNN
+F 1 "GND" H 3250 7350 50  0000 C CNN
+F 2 "" H 3250 7500 50  0001 C CNN
+F 3 "" H 3250 7500 50  0001 C CNN
+	1    3250 7500
+	-1   0    0    -1
+$EndComp
+Wire Wire Line
+	3100 7050 3500 7050
+Wire Wire Line
+	3100 7150 3500 7150
+Wire Wire Line
+	3100 7250 3250 7250
+Wire Wire Line
+	3250 7250 3250 7500
+Text Label 3500 7050 2    60   ~ 0
 SCL
-Text Label 3200 6950 0    60   ~ 0
+Text Label 3500 7150 2    60   ~ 0
 SDA
 Wire Wire Line
@@
 NoConn ~ 4200 3700
 NoConn ~ 4200 3800
+Wire Wire Line
+	3250 6850 3250 6400
+Wire Wire Line
+	3100 6850 3250 6850
+$Comp
+L VFD_Clock_LD8035-rescue:+5V #PWR013
+U 1 1 5AC42D74
+P 3250 6400
+F 0 "#PWR013" H 3250 6250 50  0001 C CNN
+F 1 "+5V" H 3250 6540 50  0000 C CNN
+F 2 "" H 3250 6400 50  0001 C CNN
+F 3 "" H 3250 6400 50  0001 C CNN
+	1    3250 6400
+	-1   0    0    -1
+$EndComp
 Wire Bus Line
 	9700 2000 9700 5750
@@
 	7700 2000 7700 5750
 Wire Bus Line
-	6600 1950 6600 3350
+	9800 3100 10550 3100
+Wire Bus Line
+	9800 1900 10550 1900
+Wire Bus Line
+	7800 5550 8700 5550
+Wire Bus Line
+	7800 4300 8700 4300
+Wire Bus Line
+	7800 3100 8700 3100
 Wire Bus Line
 	7800 1900 8750 1900
 Wire Bus Line
-	7800 3100 8700 3100
-Wire Bus Line
-	7800 4300 8700 4300
-Wire Bus Line
-	7800 5550 8700 5550
-Wire Bus Line
-	9800 1900 10550 1900
-Wire Bus Line
-	9800 3100 10550 3100
+	6600 1950 6600 3350
+$Comp
+L VFDClock_LD8035:DS3231_RTC_MODULE J3
+U 1 1 5D8B51AC
+P 2900 7050
+F 0 "J3" H 2817 6625 50  0000 C CNN
+F 1 "DS3231_RTC_MODULE" H 2817 6716 50  0000 C CNN
+F 2 "VFD:DS3231_RPi_Module" H 2900 7050 50  0001 C CNN
+F 3 "" H 2900 7050 50  0001 C CNN
+	1    2900 7050
+	-1   0    0    1
+$EndComp
 $EndSCHEMATC
