File: VFD_Clock_LD8035.sch (KiCad schematic (older format))
At the start: 22 parts, among them J1 Conn_01x04, J2 Conn_01x04, J3 DS3231_RTC_MODULE, SW1 SW_Push, SW2 SW_Push, U2 TD62783, U3 TD62783

Commit message: Add English assembly manual
Connections:
- net SDA: now also J3.4 (SDA); no longer J3.2 (NC)
Changed lines of the file:
@@
 EESchema Schematic File Version 4
 LIBS:VFD_Clock_LD8035-cache
-EELAYER 30 0
+EELAYER 29 0
 EELAYER END
 $Descr A4 11693 8268
@@
 $EndComp
 Wire Wire Line
-	3100 7050 3500 7050
-Wire Wire Line
-	3100 7150 3500 7150
-Wire Wire Line
 	3100 7250 3250 7250
 Wire Wire Line
@@
 Text Label 3500 7050 2    60   ~ 0
 SCL
-Text Label 3500 7150 2    60   ~ 0
-SDA
 Wire Wire Line
 	7800 1400 8150 1400
@@
 	-1   0    0    1
 $EndComp
+Wire Wire Line
+	3100 7050 3500 7050
+Text Label 3500 6950 2    60   ~ 0
+SDA
+Wire Wire Line
+	3100 6950 3500 6950
 Wire Bus Line
 	9700 2000 9700 5750
 Wire Bus Line
 	7700 2000 7700 5750
+Wire Bus Line
+	6600 1950 6600 3350
 Wire Bus Line
 	9800 3100 10550 3100
@@
 Wire Bus Line
 	7800 1900 8750 1900
-Wire Bus Line
-	6600 1950 6600 3350
 $EndSCHEMATC
